File: Power Distribution Board Task 6.brd (EAGLE design)
At the start: 99 x 72.1 mm, 33 parts, among them U1 MIC29300-3.3WU, U2 MIC29300-5.0WU, U3 MIC29300-12WU, X1 5566-2, X2 5566-2, X3 C-GRID-02-15-19, X4 C-GRID-02-15-19, X5 C-GRID-02-15-19, X6 C-GRID-02-15-19

Commit message: update the schematic and layout
Parts:
- C1: value (none) -> 12000uF
- C2, C3, C4: value (none) -> 47uF
- LED1: value (none) -> Green
- LED2: value (none) -> Blue
- LED3: value (none) -> Red
- LED4: value (none) -> Yellow
- R1: value (none) -> 1.2k
- R2: value (none) -> 68
- R3: value (none) -> 150
- R4: value (none) -> 560
- moved LED1 67.5 mm to (3.74, 42.3), turned to 180 degrees
- moved LED2 50.7 mm to (3.95, 31.7)
- moved R2 43.4 mm to (3.92, 27.1), turned to 180 degrees
- moved LED3 43.3 mm to (2.93, 18.7)
- moved LED4 39.4 mm to (3.27, 16.0), turned to 270 degrees
- moved R1 37.8 mm to (28.7, 49.5), turned to 180 degrees
- moved C2 37.4 mm to (28.8, 45.7), turned to 270 degrees
- moved X2 35.9 mm to (51.9, 57.6), turned to 180 degrees
- moved R3 34.1 mm to (1.43, 22.8), turned to 270 degrees
- moved X6 31.8 mm to (56.3, 34.9)
- moved R4 31.8 mm to (6.70, 19.3), turned to 270 degrees
- moved D4 31.2 mm to (35.1, 15.6), turned to 180 degrees
- moved X4 30.3 mm to (56.3, 24.1)
- moved X5 30.0 mm to (56.3, 12.2)
- moved CR4 25.9 mm to (40.1, 18.7)
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Connections:
- net N$2 renamed VSTART
- net N$3 renamed CONN
- removed net N$1: C1.2, CR1.2, R1.1, U2.2, U3.2, X1.1, X2.2
- removed net N$11: C3.1, F3.1, LED3.A, U2.4
- removed net N$14: C3.2, CR3.2, R3.1, U2.3, X4.2, X6.2
- removed net N$16: C4.1, F4.1, LED4.A, U3.4
- removed net N$19: C4.2, CR4.2, R4.1, U3.3, X5.2
- removed net N$4: CR1.1, D1.C, LED1.A, U1.1, U3.1, X2.1
- removed net N$5: C2.1, F2.1, LED2.A, U1.4
- removed net N$8: C2.2, CR2.2, R2.1, U1.3, X3.2
- new net V+: CR1.1, D1.C, LED1.A, U1.1, U2.1, U3.1, X2.1
- new net VOUT: C2.1, F2.1, LED2.A, U1.3
- new net VOUT2: C3.1, F3.1, LED3.A, U2.3
- new net VOUT3: C4.1, F4.1, LED4.A, U3.3
- net GND: now also C1.2, C2.2, C3.2, C4.2, CR1.2, CR2.2, CR3.2, CR4.2, R1.1, R2.1, R3.1, R4.1, U2.2, U3.2, X1.1, X2.2, X3.2, X4.2, X5.2, X6.2
Routing:
- net GND: track 0.00 -> 239.5 mm, vias 0 -> 6
- net V+: track 0.00 -> 123.0 mm, vias 0 -> 2
- net VOUT: track 0.00 -> 47.6 mm, vias 0 -> 2
- net VOUT2: track 0.00 -> 39.7 mm, vias 0 -> 2
- net VOUT3: track 0.00 -> 37.4 mm, vias 0 -> 2
- net N$6: track 0.00 -> 30.3 mm, vias 0 -> 2
- net N$13: track 0.00 -> 25.7 mm
- net VSTART: track 0.00 -> 22.1 mm
- net N$18: track 0.00 -> 11.3 mm
- net N$10: track 0.00 -> 7.68 mm
- net N$17: track 0.00 -> 4.81 mm
- net N$7: track 0.00 -> 4.73 mm
- net CONN: track 0.00 -> 4.11 mm
- net N$12: track 0.00 -> 3.53 mm
- net N$15: track 0.00 -> 2.67 mm
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Other:
- board size 99 x 72.1 mm -> 71.8 x 64 mm
