File: Power Distribution Board Task 6.sch (EAGLE design)
At the start: 33 parts, among them U1 MIC29300-3.3WU, U2 MIC29300-5.0WU, U3 MIC29300-12WU, X1 5566-2, X2 5566-2, X3 C-GRID-02-15-19, X4 C-GRID-02-15-19, X5 C-GRID-02-15-19, X6 C-GRID-02-15-19

Commit message: update the schematic and layout
Parts:
- C1: value (none) -> 12000uF
- C2, C3, C4: value (none) -> 47uF
- LED1: value (none) -> Green
- LED2: value (none) -> Blue
- LED3: value (none) -> Red
- LED4: value (none) -> Yellow
- R1: value (none) -> 1.2k
- R2: value (none) -> 68
- R3: value (none) -> 150
- R4: value (none) -> 560
Connections:
- net N$2 renamed VSTART
- net N$3 renamed CONN
- removed net N$1: C1.2, CR1.1, R1.1, U2.GND, U3.GND, X1-1.S, X2-2.S
- removed net N$11: C3.1, F3.1, LED3.A, U2.4
- removed net N$14: C3.2, CR3.1, R3.1, U2.OUT, X4-2.S, X6-2.S
- removed net N$16: C4.1, F4.1, LED4.A, U3.4
- removed net N$19: C4.2, CR4.1, R4.1, U3.OUT, X5-2.S
- removed net N$4: CR1.2, D1.C, LED1.A, U1.IN, U3.IN, X2-1.S
- removed net N$5: C2.1, F2.1, LED2.A, U1.4
- removed net N$8: C2.2, CR2.1, R2.1, U1.OUT, X3-2.S
- new net GND: C1.2, C2.2, C3.2, C4.2, CR1.1, CR2.1, CR3.1, CR4.1, R1.1, R2.1, R3.1, R4.1, U1.GND, U2.GND, U3.GND, X1-1.S, X2-2.S, X3-2.S, X4-2.S, X5-2.S, X6-2.S
- new net V+: CR1.2, D1.C, LED1.A, U1.IN, U2.IN, U3.IN, X2-1.S
- new net VOUT: C2.1, F2.1, LED2.A, U1.OUT
- new net VOUT2: C3.1, F3.1, LED3.A, U2.OUT
- new net VOUT3: C4.1, F4.1, LED4.A, U3.OUT
