File: 2ndNov_submission_12V_everywhere.brd (EAGLE design)
At the start: 71.8 x 64 mm, 26 parts

Commit message: finished board layout
Parts:
- moved LSP8 216.8 mm to (8.99, 46.0)
- moved VIN_12V 205.3 mm to (19.9, 55.4)
- moved LSP6 152.7 mm to (9.09, 25.1)
- moved 3A_LINE 142.6 mm to (55.5, 26.1)
- moved LSP4 120.1 mm to (8.89, 35.6)
- moved 6.25A_LINE 114.7 mm to (55.4, 38.6)
- moved GND 96.8 mm to (9.04, 55.5)
- moved 25A_LINE 84.7 mm to (55.5, 45.9)
- moved LED2 28.7 mm to (27.4, 33.7)
- moved LED3 26.7 mm to (29.3, 21.9), turned to 90 degrees
- moved LED1 22.8 mm to (26.1, 46.3), turned to 90 degrees
- moved R2 21.6 mm to (20.1, 33.6), turned to 0 degrees
- moved C3 17.5 mm to (14.4, 24.7)
- moved C2 15.9 mm to (14.4, 38.0), turned to 90 degrees
- moved R3 15.6 mm to (22.1, 22.0), turned to 0 degrees
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Routing:
- net GND: track 195.5 -> 133.1 mm, vias 6 -> 0
- net VOUT3: track 178.1 -> 145.6 mm, vias 6 -> 3
- net N$6: track 30.3 -> 2.76 mm, vias 2 -> 0
- net N$18: track 6.25 -> 24.1 mm
- net N$13: track 6.17 -> 22.8 mm
- net VSTART: track 20.8 -> 10.7 mm
- net N$20: track 2.60 -> 4.27 mm
- net N$15: track 2.67 -> 4.11 mm
- net N$17: track 4.81 -> 3.38 mm
- net N$12: track 3.53 -> 4.81 mm
- net CONN: track 4.11 -> 5.19 mm
Other:
- board size 71.8 x 64 mm -> 60.6 x 44.9 mm
