File: 2ndNov_submission_12V_everywhere.sch (EAGLE design)
At the start: 29 parts

Commit message: finished.
Parts:
- removed EXTENDERS_25A, EXTENDERS_3A, EXTENDERS_6.25A: (no value), pinhead:PINHD-2X5/90
Connections:
- removed net N$1: EXTENDERS_3A.1, EXTENDERS_3A.3, EXTENDERS_3A.5, EXTENDERS_3A.7, EXTENDERS_3A.9
- removed net N$2: EXTENDERS_3A.10, EXTENDERS_3A.2, EXTENDERS_3A.4, EXTENDERS_3A.6, EXTENDERS_3A.8
- removed net N$3: EXTENDERS_6.25A.1, EXTENDERS_6.25A.3, EXTENDERS_6.25A.5, EXTENDERS_6.25A.7, EXTENDERS_6.25A.9
- removed net N$4: EXTENDERS_6.25A.10, EXTENDERS_6.25A.2, EXTENDERS_6.25A.4, EXTENDERS_6.25A.6, EXTENDERS_6.25A.8
- removed net N$5: EXTENDERS_25A.10, EXTENDERS_25A.2, EXTENDERS_25A.4, EXTENDERS_25A.6, EXTENDERS_25A.8
- removed net N$7: EXTENDERS_25A.1, EXTENDERS_25A.3, EXTENDERS_25A.5, EXTENDERS_25A.7, EXTENDERS_25A.9
Other:
- moved on the sheet: 6.25A_LINE, C2, CR2, D2, F2, LED2, LSP4, R2
