File: 6thNov_submission_12V_everywhere.brd (EAGLE design)
At the start: 71.8 x 64 mm, 29 parts

Commit message: ERC check complete
Parts:
- EXTENDER_25A: value (none) -> 25A
- EXTENDER_3A: value (none) -> 3A
- EXTENDER_6.26A: value (none) -> 6.25A
- renumbered JP1 to EXTENDER_25A, JP2 to EXTENDER_6.26A, JP3 to EXTENDER_3A
Connections:
- removed net N$1: EXTENDER_3A.1, EXTENDER_3A.3, EXTENDER_3A.5, EXTENDER_3A.7, EXTENDER_3A.9
- removed net N$2: EXTENDER_3A.10, EXTENDER_3A.2, EXTENDER_3A.4, EXTENDER_3A.6, EXTENDER_3A.8
- removed net N$3: EXTENDER_6.26A.1, EXTENDER_6.26A.3, EXTENDER_6.26A.5, EXTENDER_6.26A.7, EXTENDER_6.26A.9
- removed net N$4: EXTENDER_6.26A.10, EXTENDER_6.26A.2, EXTENDER_6.26A.4, EXTENDER_6.26A.6, EXTENDER_6.26A.8
- removed net N$5: EXTENDER_25A.10, EXTENDER_25A.2, EXTENDER_25A.4, EXTENDER_25A.6, EXTENDER_25A.8
- removed net N$7: EXTENDER_25A.1, EXTENDER_25A.3, EXTENDER_25A.5, EXTENDER_25A.7, EXTENDER_25A.9
- net GND: now also EXTENDER_25A.1, EXTENDER_25A.3, EXTENDER_25A.5, EXTENDER_25A.7, EXTENDER_25A.9, EXTENDER_3A.1, EXTENDER_3A.3, EXTENDER_3A.5, EXTENDER_3A.7, EXTENDER_3A.9, EXTENDER_6.26A.1, EXTENDER_6.26A.3, EXTENDER_6.26A.5, EXTENDER_6.26A.7, EXTENDER_6.26A.9
- net N$13: now also EXTENDER_6.26A.10, EXTENDER_6.26A.2, EXTENDER_6.26A.4, EXTENDER_6.26A.6, EXTENDER_6.26A.8
- net N$18: now also EXTENDER_3A.10, EXTENDER_3A.2, EXTENDER_3A.4, EXTENDER_3A.6, EXTENDER_3A.8
- net VOUT3: now also EXTENDER_25A.10, EXTENDER_25A.2, EXTENDER_25A.4, EXTENDER_25A.6, EXTENDER_25A.8

Commit message: finished.
Parts:
- removed EXTENDER_25A: 25A, pinhead:2X05
- removed EXTENDER_3A: 3A, pinhead:2X05
- removed EXTENDER_6.26A: 6.25A, pinhead:2X05
- added 25A_LINE1, 3A_LINE1, 6.25A_LINE1, GND2, LSP1, LSP2: SE13, solpad:SE13
- added JP: 1, pinhead:1X02
- added JP@2: 2, pinhead:1X02
- added PIN_BANK: 1, pinhead:2X05
- added PIN_BANK@2: 2, pinhead:2X05
- moved LSP8 221.7 mm to (9.04, 50.9)
- moved VIN_12V 205.3 mm to (19.9, 55.4)
- moved LSP6 169.1 mm to (8.84, 41.5)
- moved 3A_LINE 123.0 mm to (46.1, 8.80)
- moved LSP4 117.4 mm to (8.94, 33.0)
- moved 6.25A_LINE 105.4 mm to (46.1, 32.9)
- moved GND 96.8 mm to (9.04, 55.5)
- moved 25A_LINE 75.1 mm to (46.1, 41.0)
- moved LED3 27.1 mm to (29.3, 8.40), turned to 90 degrees
- moved LED2 26.1 mm to (27.3, 27.9)
- moved LED1 22.8 mm to (26.1, 46.3), turned to 90 degrees
- moved R2 19.3 mm to (20.1, 27.8), turned to 0 degrees
- moved R3 18.9 mm to (22.1, 8.43), turned to 0 degrees
- moved C3 15.1 mm to (14.4, 11.2)
- moved F1 14.5 mm to (22.5, 51.1)
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Connections:
- new net N$1: JP@2.1, PIN_BANK@2.1, PIN_BANK@2.3, PIN_BANK@2.5, PIN_BANK@2.7, PIN_BANK@2.9
- new net N$2: JP@2.2, PIN_BANK.1, PIN_BANK.3, PIN_BANK.5, PIN_BANK.7, PIN_BANK.9
- new net N$8: JP.1, PIN_BANK.10, PIN_BANK.2, PIN_BANK.4, PIN_BANK.6, PIN_BANK.8
- new net N$9: JP.2, PIN_BANK@2.10, PIN_BANK@2.2, PIN_BANK@2.4, PIN_BANK@2.6, PIN_BANK@2.8
- net GND: now also GND2.MP, LSP1.MP, LSP2.MP; no longer EXTENDER_25A.1, EXTENDER_25A.3, EXTENDER_25A.5, EXTENDER_25A.7, EXTENDER_25A.9, EXTENDER_3A.1, EXTENDER_3A.3, EXTENDER_3A.5, EXTENDER_3A.7, EXTENDER_3A.9, EXTENDER_6.26A.1, EXTENDER_6.26A.3, EXTENDER_6.26A.5, EXTENDER_6.26A.7, EXTENDER_6.26A.9
- net N$13: now also 6.25A_LINE1.MP; no longer EXTENDER_6.26A.10, EXTENDER_6.26A.2, EXTENDER_6.26A.4, EXTENDER_6.26A.6, EXTENDER_6.26A.8
- net N$18: now also 3A_LINE1.MP; no longer EXTENDER_3A.10, EXTENDER_3A.2, EXTENDER_3A.4, EXTENDER_3A.6, EXTENDER_3A.8
- net VOUT3: now also 25A_LINE1.MP; no longer EXTENDER_25A.10, EXTENDER_25A.2, EXTENDER_25A.4, EXTENDER_25A.6, EXTENDER_25A.8
Routing:
- net VOUT3: track 178.1 -> 128.8 mm, vias 6 -> 2
- net N$6: track 30.3 -> 2.76 mm, vias 2 -> 0
- net N$8: track 0.00 -> 22.3 mm
- net N$1: track 0.00 -> 21.4 mm
- net GND: track 172.6 -> 153.1 mm, vias 6 -> 0
- net N$18: track 6.25 -> 23.9 mm
- net N$2: track 0.00 -> 17.3 mm
- net N$9: track 0.00 -> 15.9 mm
- net N$13: track 6.17 -> 21.4 mm
- net VSTART: track 20.8 -> 10.7 mm
- net N$20: track 2.60 -> 4.25 mm
- net N$15: track 2.67 -> 4.11 mm
- net N$17: track 4.81 -> 3.38 mm
- net N$12: track 3.53 -> 4.81 mm
- net CONN: track 4.11 -> 5.19 mm
Other:
- board size 71.8 x 64 mm -> 69.2 x 61.4 mm
