File: 6thNov_submission_12V_everywhere.sch (EAGLE design)
At the start: 29 parts

Commit message: ERC check complete
Parts:
- EXTENDER_25A: value (none) -> 25A
- EXTENDER_3A: value (none) -> 3A
- EXTENDER_6.26A: value (none) -> 6.25A
- renumbered JP1 to EXTENDER_25A, JP2 to EXTENDER_6.26A, JP3 to EXTENDER_3A
Connections:
- removed net N$1: EXTENDER_3A.1, EXTENDER_3A.3, EXTENDER_3A.5, EXTENDER_3A.7, EXTENDER_3A.9
- removed net N$2: EXTENDER_3A.10, EXTENDER_3A.2, EXTENDER_3A.4, EXTENDER_3A.6, EXTENDER_3A.8
- removed net N$3: EXTENDER_6.26A.1, EXTENDER_6.26A.3, EXTENDER_6.26A.5, EXTENDER_6.26A.7, EXTENDER_6.26A.9
- removed net N$4: EXTENDER_6.26A.10, EXTENDER_6.26A.2, EXTENDER_6.26A.4, EXTENDER_6.26A.6, EXTENDER_6.26A.8
- removed net N$5: EXTENDER_25A.10, EXTENDER_25A.2, EXTENDER_25A.4, EXTENDER_25A.6, EXTENDER_25A.8
- removed net N$7: EXTENDER_25A.1, EXTENDER_25A.3, EXTENDER_25A.5, EXTENDER_25A.7, EXTENDER_25A.9
- net GND: now also EXTENDER_25A.1, EXTENDER_25A.3, EXTENDER_25A.5, EXTENDER_25A.7, EXTENDER_25A.9, EXTENDER_3A.1, EXTENDER_3A.3, EXTENDER_3A.5, EXTENDER_3A.7, EXTENDER_3A.9, EXTENDER_6.26A.1, EXTENDER_6.26A.3, EXTENDER_6.26A.5, EXTENDER_6.26A.7, EXTENDER_6.26A.9
- net N$13: now also EXTENDER_6.26A.10, EXTENDER_6.26A.2, EXTENDER_6.26A.4, EXTENDER_6.26A.6, EXTENDER_6.26A.8
- net N$18: now also EXTENDER_3A.10, EXTENDER_3A.2, EXTENDER_3A.4, EXTENDER_3A.6, EXTENDER_3A.8
- net VOUT3: now also EXTENDER_25A.10, EXTENDER_25A.2, EXTENDER_25A.4, EXTENDER_25A.6, EXTENDER_25A.8

Commit message: finished.
Parts:
- removed EXTENDER_25A: 25A, pinhead:PINHD-2X5
- removed EXTENDER_3A: 3A, pinhead:PINHD-2X5
- removed EXTENDER_6.26A: 6.25A, pinhead:PINHD-2X5
- added 25A_LINE1, 3A_LINE1, 6.25A_LINE1, GND2, LSP1, LSP2: SE13, solpad:SE13
- added JP: 1, pinhead:PINHD-1X2
- added JP@2: 2, pinhead:PINHD-1X2
- added PIN_BANK: 1, pinhead:PINHD-2X5
- added PIN_BANK@2: 2, pinhead:PINHD-2X5
Connections:
- new net N$1: JP@2.1, PIN_BANK@2.1, PIN_BANK@2.3, PIN_BANK@2.5, PIN_BANK@2.7, PIN_BANK@2.9
- new net N$2: JP@2.2, PIN_BANK.1, PIN_BANK.3, PIN_BANK.5, PIN_BANK.7, PIN_BANK.9
- new net N$8: JP.1, PIN_BANK.10, PIN_BANK.2, PIN_BANK.4, PIN_BANK.6, PIN_BANK.8
- new net N$9: JP.2, PIN_BANK@2.10, PIN_BANK@2.2, PIN_BANK@2.4, PIN_BANK@2.6, PIN_BANK@2.8
- net GND: now also GND2.MP, LSP1.MP, LSP2.MP; no longer EXTENDER_25A.1, EXTENDER_25A.3, EXTENDER_25A.5, EXTENDER_25A.7, EXTENDER_25A.9, EXTENDER_3A.1, EXTENDER_3A.3, EXTENDER_3A.5, EXTENDER_3A.7, EXTENDER_3A.9, EXTENDER_6.26A.1, EXTENDER_6.26A.3, EXTENDER_6.26A.5, EXTENDER_6.26A.7, EXTENDER_6.26A.9
- net N$13: now also 6.25A_LINE1.MP; no longer EXTENDER_6.26A.10, EXTENDER_6.26A.2, EXTENDER_6.26A.4, EXTENDER_6.26A.6, EXTENDER_6.26A.8
- net N$18: now also 3A_LINE1.MP; no longer EXTENDER_3A.10, EXTENDER_3A.2, EXTENDER_3A.4, EXTENDER_3A.6, EXTENDER_3A.8
- net VOUT3: now also 25A_LINE1.MP; no longer EXTENDER_25A.10, EXTENDER_25A.2, EXTENDER_25A.4, EXTENDER_25A.6, EXTENDER_25A.8
Other:
- moved on the sheet: 3A_LINE, 6.25A_LINE, C2, C3, CR2, CR3, D2, D3, F2, F3, LED2, LED3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
